File: m2-carrier/BOOT_RESET_LED.kicad_sch (KiCad schematic)
At the start: 10 parts, among them SW2 SW_BOOT2, SW3 SW_RESET2, SW4 SW_BOOT1, SW5 SW_RESET1

Commit message: added stuff
Parts:
- removed JP4: BOOT2_JUMPER, symbol Jumper:SolderJumper_3_Open
- removed JP5: BOOT1_JUMPER, symbol Jumper:SolderJumper_3_Open
- removed JP6: RESET2_JUMPER, symbol Jumper:SolderJumper_3_Open
- removed JP7: RESET1_JUMPER, symbol Jumper:SolderJumper_3_Open
- added R26, R27: 10K, Resistor_SMD:R_0402_1005Metric, symbol Device:R_Small
Connections:
- net BUTTON_3.3VDD: now also R26.2, R27.2
- net BUTTON_RESET1: now also SW5.1, R26.1; no longer SW5.2
- net BUTTON_RESET2: now also SW3.1, R27.1; no longer SW3.2
- net GND: now also SW2.1, SW3.2, SW4.1, SW5.2
Other:
- moved on the sheet: D4, D5, SW2, SW3, SW4, SW5
