File: m2-carrier/PIN_HEADER.kicad_sch (KiCad schematic)
At the start: 2 parts, among them J4 HEADER1, J5 HEADER2

Commit message: added stuff
Connections:
- net CON_SERVO1: now also J4.15 (Pin_15); no longer J4.1 (Pin_1)
- net CON_SERVO2: now also J4.13 (Pin_13); no longer J4.3 (Pin_3)
- net CON_SERVO3: now also J4.11 (Pin_11); no longer J4.5 (Pin_5)
- net CON_SERVO4: now also J4.9 (Pin_9); no longer J4.7 (Pin_7)
- net CON_SERVO5: now also J4.7 (Pin_7); no longer J4.9 (Pin_9)
- net CON_SERVO6: now also J4.5 (Pin_5); no longer J4.11 (Pin_11)
- net CON_SERVO7: now also J4.3 (Pin_3); no longer J4.13 (Pin_13)
- net CON_SERVO8: now also J4.1 (Pin_1); no longer J4.15 (Pin_15)
Changed lines of the file:
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@@
     (effects (font (size 1.27 1.27)) (justify left))
   )
-  (hierarchical_label "CON_SERVO4" (shape input) (at 129.54 71.12 180) (fields_autoplaced)
+  (hierarchical_label "CON_SERVO4" (shape input) (at 129.54 73.66 180) (fields_autoplaced)
     (effects (font (size 1.27 1.27)) (justify right))
   )
-  (hierarchical_label "CON_SERVO1" (shape input) (at 129.54 63.5 180) (fields_autoplaced)
+  (hierarchical_label "CON_SERVO1" (shape input) (at 129.54 81.28 180) (fields_autoplaced)
     (effects (font (size 1.27 1.27)) (justify right))
   )
@@
     (effects (font (size 1.27 1.27)) (justify right))
   )
-  (hierarchical_label "CON_SERVO6" (shape input) (at 129.54 76.2 180) (fields_autoplaced)
+  (hierarchical_label "CON_SERVO6" (shape input) (at 129.54 68.58 180) (fields_autoplaced)
     (effects (font (size 1.27 1.27)) (justify right))
   )
@@
     (effects (font (size 1.27 1.27)) (justify right))
   )
-  (hierarchical_label "CON_SERVO3" (shape input) (at 129.54 68.58 180) (fields_autoplaced)
+  (hierarchical_label "CON_SERVO3" (shape input) (at 129.54 76.2 180) (fields_autoplaced)
     (effects (font (size 1.27 1.27)) (justify right))
   )
-  (hierarchical_label "CON_SERVO5" (shape input) (at 129.54 73.66 180) (fields_autoplaced)
+  (hierarchical_label "CON_SERVO5" (shape input) (at 129.54 71.12 180) (fields_autoplaced)
     (effects (font (size 1.27 1.27)) (justify right))
   )
@@
     (effects (font (size 1.27 1.27)) (justify left))
   )
-  (hierarchical_label "CON_SERVO8" (shape input) (at 129.54 81.28 180) (fields_autoplaced)
+  (hierarchical_label "CON_SERVO8" (shape input) (at 129.54 63.5 180) (fields_autoplaced)
     (effects (font (size 1.27 1.27)) (justify right))
   )
-  (hierarchical_label "CON_SERVO7" (shape input) (at 129.54 78.74 180) (fields_autoplaced)
+  (hierarchical_label "CON_SERVO7" (shape input) (at 129.54 66.04 180) (fields_autoplaced)
     (effects (font (size 1.27 1.27)) (justify right))
   )
-  (hierarchical_label "CON_SERVO2" (shape input) (at 129.54 66.04 180) (fields_autoplaced)
+  (hierarchical_label "CON_SERVO2" (shape input) (at 129.54 78.74 180) (fields_autoplaced)
     (effects (font (size 1.27 1.27)) (justify right))
   )
