File: m2-carrier/m2-carrier.kicad_pcb (KiCad board)
At the start: 4 copper layers, 49.8 x 69.6 mm, 102 parts, among them J1 2199119-4, J2 2199119-4, J3 MEM2085-00-115-00-A, J4 HEADER1, J5 HEADER2, J6 USB4120-03-C, J7 USB4120-03-C, P1 LIPO_VCC, P2 LIPO_GND, P3 ESC1_VCC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

Commit message: added stuff
Parts:
- added R26: 10K, Resistor_SMD:R_0402_1005Metric, F.Cu at (122.9, 99.8)
- added R27: 10K, Resistor_SMD:R_0402_1005Metric, F.Cu at (122.9, 100.9)
- added Y1: 27MHz, Crystal:Crystal_SMD_Abracon_ABM3-2Pin_5.0x3.2mm, B.Cu at (140.2, 87.5)
- added kibuzzard-657F4B16: G***, kibuzzard-657F4B16, F.Cu at (119.8, 91.6)
- added kibuzzard-657F4B2F: G***, kibuzzard-657F4B2F, F.Cu at (119.8, 94.4)
- added kibuzzard-657F4B96: G***, kibuzzard-657F4B96, F.Cu at (124.9, 91.6)
- added kibuzzard-657F4B96: G***, kibuzzard-657F4B96, F.Cu at (124.9, 94.4)
- added kibuzzard-657F4C86: G***, kibuzzard-657F4C86, F.Cu at (122.4, 90.1)
- added kibuzzard-657F4D51: G***, kibuzzard-657F4D51, F.Cu at (120.4, 97.0)
- added kibuzzard-657F4D6E: G***, kibuzzard-657F4D6E, F.Cu at (124.3, 97.0)
- 3V3_IO1: renamed from 3V3IO EN
- 5VREG1, JP3: renamed from 5V VREG
- C35, R23: moved to F.Cu
- moved R23 20.3 mm to (140.8, 109.3), turned to -90 degrees
- moved C35 19.2 mm to (139.4, 108.5)
- moved J3 5.50 mm to (133.2, 110.0), turned to -90 degrees
- moved C37 5.31 mm to (142.5, 97.1), turned to 90 degrees
- moved R18 3.05 mm to (127.0, 97.0), turned to 0 degrees
- moved C30 2.77 mm to (139.1, 103.1)
- moved C31 2.69 mm to (128.5, 103.4)
- moved U7 1.69 mm to (137.1, 94.1)
- moved SW1 1.61 mm to (127.2, 93.0)
- moved R17 1.51 mm to (127.0, 98.5)
- moved C32 1.50 mm to (130.8, 97.6)
- moved C33 1.50 mm to (130.8, 95.8)
- moved C34 1.50 mm to (130.8, 94.0)
- moved 3V3_IO1 1.12 mm to (122.4, 97.0)
- moved 5VREG1 1.12 mm to (122.4, 91.6)
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Connections:
- J4 pad 1: SOM_SERVO1 -> SOM_SERVO8
- J4 pad 11: SOM_SERVO6 -> SOM_SERVO3
- J4 pad 13: SOM_SERVO7 -> SOM_SERVO2
- J4 pad 15: SOM_SERVO8 -> SOM_SERVO1
- J4 pad 3: SOM_SERVO2 -> SOM_SERVO7
- J4 pad 5: SOM_SERVO3 -> SOM_SERVO6
- J4 pad 7: SOM_SERVO4 -> SOM_SERVO5
- J4 pad 9: SOM_SERVO5 -> SOM_SERVO4
- R10 pad 2: FB -> /POWER/5V_FB
- R11 pad 1: FB -> /POWER/5V_FB
- SW2 pad 1: Net-(JP4-C) -> GND
- SW3 pad 1: Net-(JP6-C) -> SOM2_RESET
- SW3 pad 2: SOM2_RESET -> GND
- SW4 pad 1: Net-(JP5-C) -> GND
- SW5 pad 1: Net-(JP7-C) -> SOM1_RESET
- SW5 pad 2: SOM1_RESET -> GND
- U3 pad 5: FB -> /POWER/5V_FB
Routing:
- net SOM_FC_5VDD: track 23.1 -> 211.5 mm, vias 0 -> 9
- net GND: track 97.6 -> 275.1 mm, vias 23 -> 36
- net SOM1_SPI0_MOSI: track 1.39 -> 112.8 mm, vias 1 -> 2
- net SOM1_SPI0_MISO: track 1.64 -> 98.1 mm, vias 1 -> 3
- net SOM_FC_3V3: track 8.91 -> 102.0 mm, vias 0 -> 4
- net SOM_9V_CAMERA: track 12.1 -> 104.1 mm, vias 0 -> 1
- net SOM_IO_3V3: track 34.8 -> 123.1 mm, vias 2 -> 4
- net SOM1_SPI0_SCK: track 1.50 -> 89.2 mm, vias 1 -> 4
- net SOM2_UART1_TX: track 0.00 -> 79.9 mm, vias 0 -> 2
- net SOM2_UART1_RX: track 0.00 -> 78.7 mm, vias 0 -> 2
- net SOM_5V_SERVO: track 8.76 -> 85.3 mm, vias 0 -> 1
- net SOM1_RESET: track 4.15 -> 78.3 mm, vias 0 -> 4
- net SOM2_I2C1_SDA: track 0.00 -> 67.1 mm, vias 0 -> 3
- net SOM_SERVO7: track 0.00 -> 66.8 mm, vias 0 -> 2
- net SOM_SERVO6: track 0.00 -> 63.6 mm, vias 0 -> 2
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- added copper zone on B.Cu, net GND
- added copper zone on In1.Cu, net GND
- added copper zone on In2.Cu, net GND
Other:
- outline, holes or cut-outs redrawn
